Commit message: servomotorTest
잘안됨 ㅠ pid 튜닝 잘해야함

File: jumpbot_description/urdf/jumpbot_v9.urdf.xacro (robot description, xacro)
@@ -5,6 +5,7 @@
 <robot name="jumpbot" xmlns:xacro="http://ros.org/wiki/xacro">
   <xacro:include filename="$(find jumpbot_description)/urdf/jumpbot_v9_shapes.urdf" />
+  <xacro:include filename="$(find jumpbot_description)/urdf/jumpbot_v9_joint.urdf" />
   <xacro:include filename="$(find jumpbot_description)/urdf/jumpbot_v9.gazebo" />
+  <xacro:include filename="$(find jumpbot_description)/urdf/jumpbot_v9.transmission" />
   <xacro:include filename="$(find jumpbot_description)/urdf/materials.xacro" />
-  <xacro:include filename="$(find jumpbot_description)/urdf/jumpbot_v9.transmission" />
 </robot>

File: jumpbot_description/urdf/jumpbot_v9_shapes.urdf (robot description, URDF)
Before this commit: robot jumpbot, 23 links, 22 joints
Joints:
- removed joint L_arm1_joint
- removed joint L_arm2_joint
- removed joint L_arm3_joint
- removed joint L_baselink_joint
- removed joint L_cam_joint
- removed joint L_leg1_L_joint
- removed joint L_leg1_R_joint
- removed joint L_leg2_joint
- removed joint L_leg3_joint
- removed joint L_motor_joint
- removed joint L_wheel_joint
- removed joint R_arm1_joint
- removed joint R_arm2_joint
- removed joint R_baselink_joint
- removed joint R_cam_joint
- removed joint R_leg1_L_joint
- removed joint R_leg1_R_joint
- removed joint R_leg2_joint
- removed joint R_leg3_joint
- removed joint R_motor_joint
- removed joint R_wheel_joint
- removed joint joint1

Commit message: 여러가지 수정
모델세분화작업중

File: jumpbot_description/urdf/jumpbot_v9.urdf.xacro (robot description, xacro)
@@ -5,4 +5,6 @@
 <robot name="jumpbot" xmlns:xacro="http://ros.org/wiki/xacro">
   <xacro:include filename="$(find jumpbot_description)/urdf/jumpbot_v9_shapes.urdf" />
+  <xacro:include filename="$(find jumpbot_description)/urdf/jumpbot_v9_arm.urdf" />
+  <xacro:include filename="$(find jumpbot_description)/urdf/jumpbot_v9_leg.urdf" />
   <xacro:include filename="$(find jumpbot_description)/urdf/jumpbot_v9_joint.urdf" />
   <xacro:include filename="$(find jumpbot_description)/urdf/jumpbot_v9.gazebo" />

File: jumpbot_description/urdf/jumpbot_v9_shapes.urdf (robot description, URDF)
Before this commit: robot jumpbot, 23 links, 0 joints
Links:
- removed link L_arm1
- removed link L_arm2
- removed link L_arm3
- removed link L_leg1_L
- removed link L_leg1_R
- removed link L_leg2
- removed link L_leg3
- removed link R_arm1
- removed link R_arm2
- removed link R_arm3
- removed link R_leg1_L
- removed link R_leg1_R
- removed link R_leg2
- removed link R_leg3
