Commit message: effort = 1 로 설정하니까 적당한 튜닝 완료
effort가 뭘까

File: jumpbot_description/urdf/jumpbot_v9_joint.urdf (robot description, URDF)
Before this commit: robot jumpbot, 0 links, 22 joints
Joints:
- joint L_arm1_joint: limit lower=-1.5707 upper=1.5707 effort=10 velocity=10 -> lower=-1.5707 upper=1.5707 effort=1 velocity=1
- joint L_arm2_joint: limit lower=-1.5707 upper=1.5707 effort=10 velocity=10 -> lower=-1.5707 upper=1.5707 effort=1 velocity=1
- joint L_arm3_joint: limit lower=-1.5707 upper=1.5707 effort=10 velocity=10 -> lower=-1.5707 upper=1.5707 effort=1 velocity=1
- joint R_arm1_joint: limit lower=-1.5707 upper=1.5707 effort=10 velocity=10 -> lower=-1.5707 upper=1.5707 effort=1 velocity=1
- joint R_arm2_joint: limit lower=-1.5707 upper=1.5707 effort=10 velocity=10 -> lower=-1.5707 upper=1.5707 effort=1 velocity=1
- joint R_arm3_joint: limit lower=-1.5707 upper=1.5707 effort=10 velocity=10 -> lower=-1.5707 upper=1.5707 effort=1 velocity=1

Commit message: weist 수정중
effort가 머냐 진짜로??

File: jumpbot_description/urdf/jumpbot_v9_joint.urdf (robot description, URDF)
Before this commit: robot jumpbot, 0 links, 22 joints
Joints:
- joint L_baselink_joint: limit lower=0 upper=0 effort=0 velocity=0 -> lower=-1.5707 upper=1.5707 effort=100 velocity=1
- joint R_baselink_joint: limit lower=0 upper=0 effort=0 velocity=0 -> lower=-1.5707 upper=1.5707 effort=100 velocity=1

Commit message: SDFormat 추가
스프링 미완성

File: jumpbot_description/urdf/jumpbot_v9_joint.urdf (robot description, URDF)
Before this commit: robot jumpbot, 0 links, 22 joints
Joints:
- joint L_baselink_joint: limit lower=-1.5707 upper=1.5707 effort=100 velocity=1 -> lower=-1.5707 upper=1.5707 effort=1 velocity=1
- joint L_leg1_L_joint: limit lower=0 upper=0 effort=0 velocity=0 -> lower=-3.141592 upper=3.141592 effort=0 velocity=0
- joint L_leg1_R_joint: limit lower=0 upper=0 effort=0 velocity=0 -> lower=-3.141592 upper=3.141592 effort=0 velocity=0
- joint L_leg2_joint: limit lower=0 upper=0 effort=0 velocity=0 -> lower=-3.141592 upper=3.141592 effort=0 velocity=0
- joint L_leg3_joint: limit lower=0 upper=0 effort=0 velocity=0 -> lower=-3.141592 upper=3.141592 effort=0 velocity=0
- joint R_baselink_joint: limit lower=-1.5707 upper=1.5707 effort=100 velocity=1 -> lower=-1.5707 upper=1.5707 effort=1 velocity=1
- joint R_leg1_L_joint: limit lower=0 upper=0 effort=0 velocity=0 -> lower=-3.141592 upper=3.141592 effort=0 velocity=0
- joint R_leg1_R_joint: limit lower=0 upper=0 effort=0 velocity=0 -> lower=-3.141592 upper=3.141592 effort=0 velocity=0
- joint R_leg2_joint: limit lower=0 upper=0 effort=0 velocity=0 -> lower=-3.141592 upper=3.141592 effort=0 velocity=0
- joint R_leg3_joint: limit lower=0 upper=0 effort=0 velocity=0 -> lower=-3.141592 upper=3.141592 effort=0 velocity=0

Commit message: model bug 수정
조인트 오류(패시브가 적용되지않는 문제 )해결
TODO: 스프링 버그 수정필수

File: jumpbot_description/urdf/jumpbot_v9_joint.urdf (robot description, URDF)
Before this commit: robot jumpbot, 0 links, 22 joints
Joints:
- joint L_leg1_L_joint: limit lower=-3.141592 upper=3.141592 effort=0 velocity=0 -> lower=-3.141592 upper=3.141592 effort=-1 velocity=-1
- joint L_leg1_R_joint: limit lower=-3.141592 upper=3.141592 effort=0 velocity=0 -> lower=-3.141592 upper=3.141592 effort=-1 velocity=-1
- joint L_leg2_joint: limit lower=-3.141592 upper=3.141592 effort=0 velocity=0 -> lower=-3.141592 upper=3.141592 effort=-1 velocity=-1
- joint L_leg3_joint: limit lower=-3.141592 upper=3.141592 effort=0 velocity=0 -> lower=-3.141592 upper=3.141592 effort=-1 velocity=-1
- joint R_leg1_L_joint: limit lower=-3.141592 upper=3.141592 effort=0 velocity=0 -> lower=-3.141592 upper=3.141592 effort=-1 velocity=-1
- joint R_leg1_R_joint: limit lower=-3.141592 upper=3.141592 effort=0 velocity=0 -> lower=-3.141592 upper=3.141592 effort=-1 velocity=-1
- joint R_leg2_joint: limit lower=-3.141592 upper=3.141592 effort=0 velocity=0 -> lower=-3.141592 upper=3.141592 effort=-1 velocity=-1
- joint R_leg3_joint: limit lower=-3.141592 upper=3.141592 effort=0 velocity=0 -> lower=-3.141592 upper=3.141592 effort=-1 velocity=-1
