Commit message: 버그 수정

File: jumpbot_description/urdf/jumpbot_v9_shapes.urdf (robot description, URDF)
Before this commit: robot jumpbot, 9 links, 0 joints
Links:
- added link imu_link; collision box size=0.001 0.001 0.001; visual box size=0.001 0.001 0.001
Joints:
- added joint imu_joint: type fixed, parent base_link, child imu_link, origin xyz=0 0 0.01
